File: ModuleV440/ModuleV440.kicad_pcb (KiCad board)
At the start: 2 copper layers, 30 x 61.4 mm, 45 parts, among them J2 AVR-ISP-6, Q1 AO3400A, U1 EL3H7(B)(TA)-G, Y1 8MHZ Ceramic Resonator

Commit message: Tidy up track
Routing:
- net SCK: track 63.5 -> 49.4 mm
Other:
- board text added: "11 Mar 2021"
- board text removed: "03 Mar 2021"
Changed lines of the file:
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@@
     (thickness 1.6)
     (drawings 46)
-    (tracks 392)
+    (tracks 379)
     (zones 0)
     (modules 45)
@@
     (effects (font (size 1 1) (thickness 0.15)) (justify mirror))
   )
-  (gr_text "03 Mar 2021" (at 113.0676 49.1626) (layer B.SilkS)
+  (gr_text "11 Mar 2021" (at 113.0676 49.1626) (layer B.SilkS)
     (effects (font (size 1 1) (thickness 0.2)) (justify right mirror))
   )
@@
   (segment (start 125.307584 70.5376) (end 123.7376 70.5376) (width 0.3) (layer F.Cu) (net 24) (status 10))
   (segment (start 125.567584 70.2776) (end 125.307584 70.5376) (width 0.3) (layer F.Cu) (net 24) (status 30))
-  (segment (start 107.739602 70.6876) (end 123.087602 70.6876) (width 0.3) (layer B.Cu) (net 24))
-  (segment (start 108.332601 70.094601) (end 107.739602 70.6876) (width 0.3) (layer B.Cu) (net 24))
-  (segment (start 106.630599 68.392599) (end 107.734601 68.392599) (width 0.3) (layer B.Cu) (net 24))
-  (segment (start 107.734601 68.392599) (end 108.332601 68.990599) (width 0.3) (layer B.Cu) (net 24))
-  (segment (start 106.032599 68.990599) (end 106.630599 68.392599) (width 0.3) (layer B.Cu) (net 24))
-  (segment (start 108.332601 68.990599) (end 108.332601 70.094601) (width 0.3) (layer B.Cu) (net 24))
-  (segment (start 106.032599 70.094601) (end 106.032599 68.990599) (width 0.3) (layer B.Cu) (net 24))
-  (segment (start 105.199602 70.6876) (end 106.625598 70.6876) (width 0.3) (layer B.Cu) (net 24))
-  (segment (start 105.792601 68.990599) (end 105.792601 70.094601) (width 0.3) (layer B.Cu) (net 24))
-  (segment (start 104.090599 68.392599) (end 105.194601 68.392599) (width 0.3) (layer B.Cu) (net 24))
-  (segment (start 103.492599 68.990599) (end 104.090599 68.392599) (width 0.3) (layer B.Cu) (net 24))
-  (segment (start 104.085598 70.6876) (end 103.492599 70.094601) (width 0.3) (layer B.Cu) (net 24))
-  (segment (start 102.9376 69.9476) (end 103.6776 70.6876) (width 0.3) (layer B.Cu) (net 24))
-  (segment (start 102.9376 68.7076) (end 102.9376 69.9476) (width 0.3) (layer B.Cu) (net 24))
-  (segment (start 105.194601 68.392599) (end 105.792601 68.990599) (width 0.3) (layer B.Cu) (net 24))
-  (segment (start 123.087602 70.6876) (end 123.337601 70.937599) (width 0.3) (layer B.Cu) (net 24))
-  (segment (start 103.6776 70.6876) (end 104.085598 70.6876) (width 0.3) (layer B.Cu) (net 24))
-  (segment (start 105.792601 70.094601) (end 105.199602 70.6876) (width 0.3) (layer B.Cu) (net 24))
-  (segment (start 123.337601 70.937599) (end 123.7376 70.5376) (width 0.3) (layer B.Cu) (net 24))
-  (segment (start 106.625598 70.6876) (end 106.032599 70.094601) (width 0.3) (layer B.Cu) (net 24))
-  (segment (start 103.492599 70.094601) (end 103.492599 68.990599) (width 0.3) (layer B.Cu) (net 24))
-  (segment (start 104.6426 67.0026) (end 102.9376 68.7076) (width 0.3) (layer B.Cu) (net 24) (status 10))
   (segment (start 114.117414 80.311817) (end 114.205091 80.399494) (width 0.3) (layer B.Cu) (net 24))
   (segment (start 114.205091 80.437593) (end 113.836818 80.805866) (width 0.3) (layer B.Cu) (net 24))
@@
   (segment (start 122.1676 78.2876) (end 126.1776 74.2776) (width 0.3) (layer B.Cu) (net 24))
   (segment (start 115.7676 78.2876) (end 122.1676 78.2876) (width 0.3) (layer B.Cu) (net 24))
+  (segment (start 104.6426 67.0026) (end 105.2826 67.0026) (width 0.3) (layer B.Cu) (net 24))
+  (segment (start 105.8776 68.2376) (end 104.6426 67.0026) (width 0.25) (layer B.Cu) (net 24))
+  (segment (start 105.9176 68.2376) (end 105.8776 68.2376) (width 0.25) (layer B.Cu) (net 24))
+  (segment (start 123.5876 70.6876) (end 123.7376 70.5376) (width 0.3) (layer B.Cu) (net 24))
+  (segment (start 108.7176 70.2376) (end 109.1676 70.6876) (width 0.3) (layer B.Cu) (net 24))
+  (segment (start 108.073601 68.2376) (end 108.7176 68.881599) (width 0.3) (layer B.Cu) (net 24))
+  (segment (start 105.9176 68.2376) (end 108.073601 68.2376) (width 0.3) (layer B.Cu) (net 24))
+  (segment (start 108.7176 68.881599) (end 108.7176 70.2376) (width 0.3) (layer B.Cu) (net 24))
+  (segment (start 109.1676 70.6876) (end 123.5876 70.6876) (width 0.3) (layer B.Cu) (net 24))
   (via (at 110.1176 100.0976) (size 0.8) (drill 0.4) (layers F.Cu B.Cu) (net 25))
   (segment (start 109.3926 103.4876) (end 109.6676 103.7626) (width 0.5) (layer F.Cu) (net 25) (status 30))
